File: Motor_Driver/untitled.kicad_sch (KiCad schematic)
At the start: 20 parts, among them J1 USB_C_Receptacle_USB2.0_16P, J2 12V_Terminal, J3 3.3V_Terminal, J4 Conn_01x03_Pin, J5 Conn_01x03_Pin, J6 Conn_01x03_Pin, Q1 PMOS, Q2 PMOS, U2 USBLC6-2SC6, U3 SN65HVD230

Commit message: Schematic Changes 90% done
Parts:
- removed D6: D_TVS, symbol Device:D_TVS
- removed J5: Conn_01x03_Pin, symbol Connector:Conn_01x03_Pin
- added C20, C21, C24, C25: C, symbol Device:C
- added C22: 470μF, symbol Device:C
- added C23, C26, C27: 4.7nF, symbol Device:C
- added C28: 100nF, symbol Device:C
- added D16: SMBJ15CA, symbol Device:D_Zener
- added D6: PESD3V3S1UL, Diode_SMD:D_SOD-882, symbol Diode:PESD3V3S1UL
- added D7: PESD5V0S1UL, Diode_SMD:D_SOD-882, symbol Diode:PESD5V0S1UL
- added F1, F2: Polyfuse, symbol Device:Polyfuse
- added J5: Conn_01x04_Pin, symbol Connector:Conn_01x04_Pin
- added R28, R29: 4.7k, symbol Device:R
- added R30: 10k, symbol Device:R
- added R31, R32: 1k, symbol Device:R
- added R7: 120R, symbol Device:R
- added U6, U7: TMP1075D, Package_SO:SO-8_3.9x4.9mm_P1.27mm, symbol Sensor_Temperature:TMP1075D
- added U8, U9: PMCS1101A1BQDR, TMCS1101:D0008A_N, symbol TMCS1101:PMCS1101A1BQDR
Connections:
- net GND: now also U3.8 (Rs), C20.1, C21.1, C22.1, C23.2, C24.1, C25.1, C26.2, C27.1, C28.1, D16.2 (A), D6.2 (A), D7.2 (A), J5.2 (Pin_2), U6.4 (GND), U6.5 (A2), U6.6 (A1), U6.7 (A0), U7.4 (GND), U7.5 (A2), U7.6 (A1), U8.5 (GND), U8.6 (NC), U9.5 (GND), U9.6 (NC)
- net SCL: now also R29.2, U6.2 (SCL), U7.2 (SCL); no longer D2.1 (K), J6.3 (Pin_3)
- net SDA: now also R28.2, U6.1 (SDA), U7.1 (SDA); no longer D3.1 (K), J6.2 (Pin_2)
- net at J4.1 (Pin_1), U3.7 (CANH): now also D7.1 (K), R7.1
- net at J4.2 (Pin_2), U3.6 (CANL): now also R7.2
- net CAN_TX: now reaches U3.1 (D)
- net CAN_RX: now reaches U3.4 (R)
- net RP_12V renamed +12V
- net +12V: now also C22.2, D16.1 (K), F1.1, F2.1
- net RP_3.3V renamed +3V3
- net +3V3: now also C20.2, C21.2, C24.2, C25.2, C27.2, C28.2, D6.1 (K), J5.1 (Pin_1), R28.1, R29.1, R30.1, U6.8 (V+), U7.7 (A0), U7.8 (V+), U8.8 (VS), U9.8 (VS)
- net RX renamed UART_RX
- net UART_RX: now also J5.4 (Pin_4)
- net TX renamed UART_TX
- net UART_TX: now also J5.3 (Pin_3)
- new net: F2.2, U9.1 (IS+), U9.2 (IS+)
- new net: R32.1, U9.7 (OUT)
- new net: R31.1, U8.7 (OUT)
- new net: F1.2, U8.1 (IS+), U8.2 (IS+)
- new net +12V_M1: U8.3 (IS-), U8.4 (IS-)
- new net +12V_M2: U9.3 (IS-), U9.4 (IS-)
- new net I2C_SCL: D2.1 (K), J6.3 (Pin_3)
- new net I2C_SDA: D3.1 (K), J6.2 (Pin_2)
- new net M1_I_SENSE: C23.1, R31.2
- new net M2_I_SENSE: C26.1, R32.2
- new net TEMP_ALERT: R30.2, U6.3 (ALERT), U7.3 (ALERT)
- no-connect marks 4 -> 5
Other:
- added sheet H_Bridge (h_bridge.kicad_sch)
- note added: "12V reverse polarity plus bulk capicitors and TVS"
- note added: "3.3V reverse polarity plus bulk capacitors and TVS"
- note added: "CAN connector + CAN transciever"
- note added: "Current Sensing ICs"
- note added: "I2C Connector"
- note added: "Motor 1, Address 0x48"
- note added: "Motor 2, Address 0x49"
- note added: "Power Inputs"
- note added: "Temperature sensors"
- note added: "To MCU"
- note added: "USB C connector + ESD connector"
- note added: "Uart Connector"
- moved on the sheet: D1, D2, D3, D4, D5, J1, J4, J6, Q1, Q2, R3, R4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
