File: Motor_Driver/h_bridge.kicad_sch (KiCad schematic)
At the start: 52 parts, among them M1 Motor_DC, M2 Motor_DC, Q10 PMOS, Q11 CSD18540Q5B, Q12 SQJ407EP, Q13 CSD18540Q5B, Q14 MMBT3904, Q3 CSD18540Q5B, Q4 CSD18540Q5B, Q5 SQJ407EP, Q6 PMOS, Q7 MMBT3904, Q8 MMBT3904, Q9 MMBT3904, U4 UCC27524D, U5 UCC27524D

Commit message: Potential Finished Schematic Before Placements
Connections:
- net M1_EN_A: no longer names the net of U4.1 (ENA)
- net M1_EN_B: no longer names the net of U4.8 (ENB)
- net M2_EN_A: no longer names the net of U5.1 (ENA)
- net M2_EN_B: no longer names the net of U5.8 (ENB)
- no-connect marks 0 -> 4
Changed lines of the file:
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@@
 		(color 0 0 0 0)
+	)
+	(no_connect
+		(at 292.1 190.5)
+	)
+	(no_connect
+		(at 102.87 190.5)
+	)
+	(no_connect
+		(at 292.1 180.34)
+	)
+	(no_connect
+		(at 102.87 180.34)
 	)
 	(wire
@@
 		)
 	)
-	(global_label "M2_EN_B"
-		(shape input)
-		(at 292.1 190.5 180)
-		(fields_autoplaced yes)
-		(effects
-			(font
-				(size 1.27 1.27)
-			)
-			(justify right)
-		)
-		(property "Intersheetrefs" "${INTERSHEET_REFS}"
-			(at 280.7692 190.5 0)
-			(hide yes)
-			(show_name no)
-			(do_not_autoplace no)
-			(effects
-				(font
-					(size 1.27 1.27)
-				)
-				(justify right)
-			)
-		)
-	)
-	(global_label "M1_EN_A"
-		(shape input)
-		(at 102.87 180.34 180)
-		(fields_autoplaced yes)
-		(effects
-			(font
-				(size 1.27 1.27)
-			)
-			(justify right)
-		)
-		(property "Intersheetrefs" "${INTERSHEET_REFS}"
-			(at 91.7206 180.34 0)
-			(hide yes)
-			(show_name no)
-			(do_not_autoplace no)
-			(effects
-				(font
-					(size 1.27 1.27)
-				)
-				(justify right)
-			)
-		)
-	)
 	(global_label "M1_PWM_A"
 		(shape input)
@@
 		)
 	)
-	(global_label "M2_EN_A"
-		(shape input)
-		(at 292.1 180.34 180)
-		(fields_autoplaced yes)
-		(effects
-			(font
-				(size 1.27 1.27)
-			)
-			(justify right)
-		)
-		(property "Intersheetrefs" "${INTERSHEET_REFS}"
-			(at 280.9506 180.34 0)
-			(hide yes)
-			(show_name no)
-			(do_not_autoplace no)
-			(effects
-				(font
-					(size 1.27 1.27)
-				)
-				(justify right)
-			)
-		)
-	)
 	(global_label "M1_P_A_ON"
 		(shape input)
@@
 			(hide yes)
 			(show_name no)
-			(do_not_autoplace no)
-			(effects
-				(font
-					(size 1.27 1.27)
-				)
-				(justify right)
-			)
-		)
-	)
-	(global_label "M1_EN_B"
-		(shape input)
-		(at 102.87 190.5 180)
-		(fields_autoplaced yes)
-		(effects
-			(font
-				(size 1.27 1.27)
-			)
-			(justify right)
-		)
-		(property "Intersheetrefs" "${INTERSHEET_REFS}"
-			(at 91.5392 190.5 0)
-			(hide yes)
-			(show_name no)

Commit message: Hopefully fully finished schematic. Ready for PCB placement.
Parts:
- removed M1, M2: Motor_DC, symbol Motor:Motor_DC
- added J8, J9: Screw_Terminal_01x02, TerminalBlock:TerminalBlock_MaiXu_MX126-5.0-02P_1x02_P5.00mm, symbol Connector:Screw_Terminal_01x02
- added TP3, TP4: TestPoint, TestPoint:TestPoint_Pad_D1.5mm, symbol Connector:TestPoint
- C12, C18: value C -> 0.1μF; footprint (none) -> Capacitor_SMD:C_0805_2012Metric
- C13, C14, C17, C19: footprint (none) -> Capacitor_SMD:C_0805_2012Metric
- C15, C16: footprint (none) -> Capacitor_SMD:CP_Elec_8x10.5
- D10, D11, D12, D15: footprint (none) -> Diode_SMD:D_SOD-123
- D13, D14, D8, D9: footprint (none) -> Package_TO_SOT_SMD:TO-277A
- Q10, Q6: value PMOS -> SQJ407EP; footprint (none) -> Package_SO:PowerPAK_SO-8_Single
- Q11, Q13, Q3, Q4: footprint (none) -> Package_TO_SOT_SMD:TDSON-8-1
- Q12, Q5: footprint (none) -> Package_SO:PowerPAK_SO-8_Single
- R10, R11, R12, R13, R14, R15, R16, R17, R18, R19, R20, R21, R22, R23, R24, R25, R26, R27, R8, R9: footprint (none) -> Resistor_SMD:R_0805_2012Metric
Connections:
- net +12V_M1: now also TP3.1
- net +12V_M2: now also TP4.1
- net M1_OUT2: now reaches C12.2, D9.2 (A), Q4.1 (D), Q5.1 (D)
- net M1_OUT2: now also J8.2 (Pin_2)
- net M2_OUT1: now reaches C18.1, D13.2 (A), Q10.1 (D), Q11.1 (D)
- net M2_OUT1: now also J9.1 (Pin_1)
- net M2_OUT2: now reaches C18.2, D14.2 (A), Q12.1 (D), Q13.1 (D)
- net M2_OUT2: now also J9.2 (Pin_2)
- net M1_OUT1: now reaches C12.1, D8.2 (A), Q3.1 (D), Q6.1 (D)
- net M1_OUT1: now also J8.1 (Pin_1)
