File: Motor_Driver/Motor_Driver.kicad_sch (KiCad schematic)
At the start: 14 parts, among them U1 RP2040

Commit message: Schematic Changes 90% done
Connections:
- net +1V1: now also U1.45 (VREG_VOUT)
Other:
- sheet sheet1.kicad_sch renamed connections.kicad_sch
- sheet connections.kicad_sch: file untitled.kicad_sch -> connections.kicad_sch
- note added: "Bulk Capacitors"
- moved on the sheet: C1, C10, C11, C2, C3, C4, C5, C6, C7, C8, C9, R1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

Commit message: Potential Finished Schematic Before Placements
Connections:
- net M1_P_A_ON: now reaches U1.11 (GPIO8)
- net M1_P_B_ON: now reaches U1.12 (GPIO9)
- net M1_PWM_A: now reaches U1.13 (GPIO10)
- net M1_PWM_B: now reaches U1.14 (GPIO11)
- net M2_PWM_A: now reaches U1.15 (GPIO12)
- net M2_PWM_B: now reaches U1.16 (GPIO13)
- net M2_P_A_ON: now reaches U1.17 (GPIO14)
- net M2_P_B_ON: now reaches U1.18 (GPIO15)
- net UART_TX: now reaches U1.2 (GPIO0)
- net STATUS_LED: now reaches U1.27 (GPIO16)
- net UART_RX: now reaches U1.3 (GPIO1)
- net SPI_MISO: now reaches U1.31 (GPIO20)
- net SPI_CS: now reaches U1.32 (GPIO21)
- net SPI_SCK: now reaches U1.34 (GPIO22)
- net SPI_MOSI: now reaches U1.35 (GPIO23)
- net M1_ISENSE: now reaches U1.38 (GPIO26/ADC0)
- net M2_ISENSE: now reaches U1.39 (GPIO27/ADC1)
- net CAN_TX: now reaches U1.4 (GPIO2)
- net CAN_RX: now reaches U1.5 (GPIO3)
- net SDA: now reaches U1.6 (GPIO4)
- net SCL: now reaches U1.7 (GPIO5)
- net TEMP_ALERT: now reaches U1.8 (GPIO6)
- no-connect marks 0 -> 13
Other:
- note added: "RP2040 MicroController"
- moved on the sheet: C1, C10, C11, C2, C3, C4, C5, C6, C7, C8, C9

Commit message: Hopefully fully finished schematic. Ready for PCB placement.
Parts:
- added C29, C30: 100nF, Capacitor_SMD:C_0805_2012Metric, symbol Device:C
- added C31, C32: 15p, Capacitor_SMD:C_0805_2012Metric, symbol Device:C
- added D21, D22, D23: LED, LED_SMD:LED_0805_2012Metric, symbol Device:LED
- added R33, R35: 1k, Resistor_SMD:R_0805_2012Metric, symbol Device:R
- added R34: 10k, Resistor_SMD:R_0805_2012Metric, symbol Device:R
- added R36, R37: 1K, Resistor_SMD:R_0805_2012Metric, symbol Device:R
- added R38: 4.7K, Resistor_SMD:R_0805_2012Metric, symbol Device:R
- added SW1: SW_Push, Button_Switch_THT:SW_PUSH_6mm, symbol Switch:SW_Push
- added SW2: BOOTSEL, Button_Switch_THT:SW_PUSH_6mm, symbol Switch:SW_Push
- added TP5, TP6, TP7, TP8: TestPoint, TestPoint:TestPoint_Pad_D1.5mm, symbol Connector:TestPoint
- added U10: W25Q16JVSS, Package_SO:SOIC-8_5.3x5.3mm_P1.27mm, symbol Memory_Flash:W25Q16JVSS
- added U11: TPS3839DBZ, Package_TO_SOT_SMD:SOT-23, symbol Power_Supervisor:TPS3839DBZ
- added Y1: 12MHz, Crystal:Crystal_SMD_3225-4Pin_3.2x2.5mm, symbol Device:Crystal_GND24
- C1, C10, C11, C2, C3, C4, C5, C6, C7, C8, C9: footprint (none) -> Capacitor_SMD:C_0805_2012Metric
- R1, R2: footprint (none) -> Resistor_SMD:R_0805_2012Metric
Connections:
- net +3V3: now also C29.1, C30.1, R34.1, R37.1, TP5.1, U10.8 (VCC), U11.3 (VDD)
- net GND: now also C29.2, C30.2, C31.1, C32.1, D21.1 (K), D22.1 (K), D23.1 (K), SW1.1, SW2.1, TP6.1, TP7.1, U10.4 (GND), U11.1 (GND), Y1.2 (G), Y1.4 (G)
- net STATUS_LED: now also R36.1
- net XIN: now reaches U1.20 (XIN)
- net XIN: now also C32.2, Y1.1
- net XOUT: now reaches U1.21 (XOUT)
- net XOUT: now also C31.2, Y1.3
- net at U1.26 (RUN): now also R34.2, R35.2, SW1.2
- net 12V_SENSE: now reaches U1.40 (GPIO28/ADC2)
- net RP_SCLK: now reaches U1.52 (QSPI_SCLK)
- net RP_SCLK: now also U10.6 (CLK)
- net RP_QSPI_SS: now reaches U1.56 (~{QSPI_SS})
- net RP_QSPI_SS: now also R33.1, U10.1 (~{CS})
- net M1_ISENSE renamed M1_I_SENSE
- net M2_ISENSE renamed M2_I_SENSE
- new net: R33.2, SW2.2
- new net: D21.2 (A), R36.2
- new net: D22.2 (A), R37.2
- new net: R35.1, U11.2 (~{RESET})
- new net: D23.2 (A), R38.2
- new net +12V: R38.1, TP8.1
Other:
- note added: "12V Power Flag"
- note added: "3.3 Power Flag"
- note added: "Crystal"
- note added: "Flash Memory"
- note added: "Status LED"
- moved on the sheet: C1, C10, C11, C2, C3, C4, C5, C6, C7, C8, C9, R1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

Commit message: Several Bug fixes
Connections:
- net USB_D+ renamed Clean_USB_D+
- net USB_D- renamed Clean_USB_D-
- no-connect marks 13 -> 17
Changed lines of the file:
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@@
 		(color 0 0 0 0)
 	)
+	(junction
+		(at 340.36 27.94)
+		(diameter 0)
+		(color 0 0 0 0)
+	)
+	(no_connect
+		(at 140.97 153.67)
+	)
 	(no_connect
 		(at 195.58 176.53)
@@
 	)
 	(no_connect
+		(at 140.97 161.29)
+	)
+	(no_connect
 		(at 140.97 189.23)
 	)
@@
 	)
 	(no_connect
+		(at 140.97 158.75)
+	)
+	(no_connect
 		(at 39.37 248.92)
 	)
@@
 		(at 195.58 158.75)
 	)
+	(no_connect
+		(at 140.97 156.21)
+	)
 	(wire
 		(pts
@@
 	(wire
 		(pts
-			(xy 306.07 46.99) (xy 306.07 50.8)
-		)
-		(stroke
-			(width 0)
-			(type default)
-		)
-	)
-	(wire
-		(pts
 			(xy 177.8 250.19) (xy 182.88 250.19)
 		)
@@
 	(wire
 		(pts
+			(xy 317.5 26.67) (xy 317.5 29.21)
+		)
+		(stroke
+			(width 0)
+			(type default)
+		)
+	)
+	(wire
+		(pts
 			(xy 332.74 57.15) (xy 332.74 58.42)
 		)
@@
 	(wire
 		(pts
+			(xy 306.07 46.99) (xy 306.07 48.26)
+		)
+		(stroke
+			(width 0)
+			(type default)
+		)
+	)
+	(wire
+		(pts
 			(xy 193.04 267.97) (xy 194.31 267.97)
 		)
@@
 	(wire
 		(pts
-			(xy 317.5 26.67) (xy 317.5 29.21)
-		)
-		(stroke
-			(width 0)
-			(type default)
-		)
-	)
-	(wire
-		(pts
 			(xy 190.5 233.68) (xy 194.31 233.68)
 		)
@@
 		)
 	)
-	(global_label "USB_D+"
+	(global_label "Clean_USB_D+"
 		(shape input)
 		(at 109.22 143.51 180)
@@
 		)
 		(property "Intersheetrefs" "${INTERSHEET_REFS}"
-			(at 98.6148 143.51 0)
+			(at 92.3254 143.51 0)
 			(hide yes)
 			(show_name no)
@@
 		)
 	)
-	(global_label "USB_D-"
+	(global_label "Clean_USB_D-"
 		(shape input)
 		(at 109.22 135.89 180)
@@
 		)
 		(property "Intersheetrefs" "${INTERSHEET_REFS}"
-			(at 98.6148 135.89 0)
+			(at 92.3254 135.89 0)
 			(hide yes)
 			(show_name no)
@@
 	(symbol
 		(lib_id "power:GND")
-		(at 306.07 50.8 0)
+		(at 306.07 48.26 0)
 		(unit 1)
 		(body_style 1)
@@
 		(fields_autoplaced yes)
 		(property "Reference" "#PWR01"
-			(at 306.07 57.15 0)
+			(at 306.07 54.61 0)
 			(hide yes)
 			(show_name no)
@@
 		)
 		(property "Value" "GND"
-			(at 306.07 55.88 0)
+			(at 306.07 53.34 0)
 			(show_name no)
 			(do_not_autoplace no)
@@
 		)
 		(property "Footprint" ""
-			(at 306.07 50.8 0)
+			(at 306.07 48.26 0)
 			(hide yes)
 			(show_name no)
@@
 		)
 		(property "Datasheet" ""
-			(at 306.07 50.8 0)
+			(at 306.07 48.26 0)
 			(hide yes)
 			(show_name no)
@@
 		)
 		(property "Description" "Power symbol creates a global label with name \"GND\" , ground"
-			(at 306.07 50.8 0)
+			(at 306.07 48.26 0)
 			(hide yes)
 			(show_name no)
@@
 					(unit 1)
 				)
+			)
+		)
+	)
+	(symbol
+		(lib_id "power:PWR_FLAG")
+		(at 340.36 27.94 270)
+		(unit 1)
+		(body_style 1)
+		(exclude_from_sim no)
+		(in_bom yes)
+		(on_board yes)
+		(in_pos_files yes)
+		(dnp no)
+		(fields_autoplaced yes)
+		(property "Reference" "#FLG02"
+			(at 342.265 27.94 0)
+			(hide yes)
+			(show_name no)
+			(do_not_autoplace no)
+			(effects
+				(font
+					(size 1.27 1.27)
+				)
+			)
+		)
+		(property "Value" "PWR_FLAG"
+			(at 344.17 27.9399 90)
+			(show_name no)
+			(do_not_autoplace no)
+			(effects
+				(font
+					(size 1.27 1.27)
+				)
+				(justify left)
+			)
+		)
+		(property "Footprint" ""
+			(at 340.36 27.94 0)
+			(hide yes)
+			(show_name no)
+			(do_not_autoplace no)
+			(effects
+				(font
+					(size 1.27 1.27)
+				)
+			)
+		)
+		(property "Datasheet" ""
+			(at 340.36 27.94 0)
+			(hide yes)
+			(show_name no)
+			(do_not_autoplace no)
+			(effects
+				(font
+					(size 1.27 1.27)
+				)
+			)
+		)
+		(property "Description" "Special symbol for telling ERC where power comes from"
+			(at 340.36 27.94 0)
+			(hide yes)
+			(show_name no)
+			(do_not_autoplace no)
+			(effects
+				(font
+					(size 1.27 1.27)
+				)
+			)
+		)
+		(pin "1"
+		)
+		(instances
+			(project "Motor_Driver"
+				(path "/73a47b03-d134-4703-ba74-88b80604f77f"
+					(reference "#FLG02")
+					(unit 1)
+				)
