File: Motor_Driver/connections.kicad_sch (KiCad schematic)
At the start: 43 parts, among them J1 USB_C_Receptacle_USB2.0_16P, J2 12V_Terminal, J3 3.3V_Terminal, J4 Conn_01x03_Pin, J5 Conn_01x04_Pin, J6 Conn_01x03_Pin, Q1 PMOS, Q2 PMOS, U2 USBLC6-2SC6, U3 SN65HVD230, U6 TMP1075D, U7 TMP1075D, U8 PMCS1101A1BQDR, U9 PMCS1101A1BQDR

Commit message: Potential Finished Schematic Before Placements
Parts:
- added D17, D18, D19, D20: PESD5V0S1UL, Diode_SMD:D_SOD-882, symbol Diode:PESD5V0S1UL
- added J7: Conn_01x06_Pin, symbol Connector:Conn_01x06_Pin
Connections:
- net +3V3: now also J7.2 (Pin_2)
- net GND: now also D17.2 (A), D18.2 (A), D19.2 (A), D20.2 (A), J7.1 (Pin_1)
- new net SPI_CS: D17.1 (K), J7.6 (Pin_6)
- new net SPI_MISO: D18.1 (K), J7.5 (Pin_5)
- new net SPI_MOSI: D19.1 (K), J7.4 (Pin_4)
- new net SPI_SCK: D20.1 (K), J7.3 (Pin_3)
Other:
- note added: "SPI Connector"
- moved on the sheet: C20, C21, C22, C23, C24, C25, C26, C27, C28, D1, D16, D2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

Commit message: Hopefully fully finished schematic. Ready for PCB placement.
Parts:
- added C33: 100nF, Capacitor_SMD:C_0805_2012Metric, symbol Device:C
- added R39: 100k, Resistor_SMD:R_0805_2012Metric, symbol Device:R
- added R40: 22k, Resistor_SMD:R_0805_2012Metric, symbol Device:R
- added TP1, TP2: TestPoint, TestPoint:TestPoint_Pad_D1.5mm, symbol Connector:TestPoint
- C20, C21, C23, C24, C25, C26, C27, C28: footprint (none) -> Capacitor_SMD:C_0805_2012Metric
- C22: footprint (none) -> Capacitor_SMD:CP_Elec_10x10.5
- D1: footprint (none) -> Diode_SMD:D_SOD-123
- D16: footprint (none) -> Diode_SMD:D_SMB
- F1, F2: footprint (none) -> MotorDriver:PTC_FUSE
- J1: footprint (none) -> Connector_USB:USB_C_Receptacle_GCT_USB4105-xx-A_16P_TopMnt_Horizontal
- J2, J3: footprint (none) -> TerminalBlock:TerminalBlock_MaiXu_MX126-5.0-02P_1x02_P5.00mm
- J4, J6: footprint (none) -> Connector_JST:JST_XH_B3B-XH-A_1x03_P2.50mm_Vertical
- J5: footprint (none) -> Connector_JST:JST_XH_B4B-XH-A_1x04_P2.50mm_Vertical
- J7: footprint (none) -> Connector_JST:JST_XH_B6B-XH-A_1x06_P2.50mm_Vertical
- Q1, Q2: footprint (none) -> Package_SO:PowerPAK_SO-8_Single
- R28, R29, R3, R30, R31, R32, R4, R5, R6, R7: footprint (none) -> Resistor_SMD:R_0805_2012Metric
Connections:
- net +12V: now also R39.1
- net GND: now also C33.2, R40.2
- net Raw_12V: now also TP1.1
- net Raw_3.3V: now also TP2.1
- new net 12V_SENSE: C33.1, R39.2, R40.1
Other:
- note added: "Voltage Sense of 12V"

Commit message: Several Bug fixes
Parts:
- C20, C21, C24, C25: value C -> 100nF
Changed lines of the file:
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@@
 	)
 	(junction
+		(at 179.07 50.8)
+		(diameter 0)
+		(color 0 0 0 0)
+	)
+	(junction
 		(at 156.21 50.8)
 		(diameter 0)
@@
 	)
 	(junction
+		(at 62.23 38.1)
+		(diameter 0)
+		(color 0 0 0 0)
+	)
+	(junction
 		(at 49.53 236.22)
 		(diameter 0)
@@
 		)
 	)
-	(label "USB_D-"
-		(at 77.47 118.11 0)
-		(effects
-			(font
-				(size 1.27 1.27)
-			)
-			(justify left bottom)
-		)
-	)
-	(label "USB_D+"
-		(at 77.47 115.57 0)
-		(effects
-			(font
-				(size 1.27 1.27)
-			)
-			(justify left bottom)
-		)
-	)
 	(global_label "SPI_SCK"
 		(shape input)
@@
 		)
 	)
+	(global_label "USB_D-"
+		(shape input)
+		(at 77.47 118.11 180)
+		(fields_autoplaced yes)
+		(effects
+			(font
+				(size 1.27 1.27)
+			)
+			(justify right)
+		)
+		(property "Intersheetrefs" "${INTERSHEET_REFS}"
+			(at 66.8648 118.11 0)
+			(hide yes)
+			(show_name no)
+			(do_not_autoplace no)
+			(effects
+				(font
+					(size 1.27 1.27)
+				)
+				(justify right)
+			)
+		)
+	)
+	(global_label "USB_D+"
+		(shape input)
+		(at 77.47 115.57 180)
+		(fields_autoplaced yes)
+		(effects
+			(font
+				(size 1.27 1.27)
+			)
+			(justify right)
+		)
+		(property "Intersheetrefs" "${INTERSHEET_REFS}"
+			(at 66.8648 115.57 0)
+			(hide yes)
+			(show_name no)
+			(do_not_autoplace no)
+			(effects
+				(font
+					(size 1.27 1.27)
+				)
+				(justify right)
+			)
+		)
+	)
 	(global_label "I2C_SDA"
 		(shape input)
@@
 	)
 	(symbol
+		(lib_id "power:PWR_FLAG")
+		(at 62.23 38.1 270)
+		(unit 1)
+		(body_style 1)
+		(exclude_from_sim no)
+		(in_bom yes)
+		(on_board yes)
+		(in_pos_files yes)
+		(dnp no)
+		(fields_autoplaced yes)
+		(property "Reference" "#FLG01"
+			(at 64.135 38.1 0)
+			(hide yes)
+			(show_name no)
+			(do_not_autoplace no)
+			(effects
+				(font
+					(size 1.27 1.27)
+				)
+			)
+		)
+		(property "Value" "PWR_FLAG"
+			(at 66.04 38.0999 90)
+			(show_name no)
+			(do_not_autoplace no)
+			(effects
+				(font
+					(size 1.27 1.27)
+				)
+				(justify left)
+			)
+		)
+		(property "Footprint" ""
+			(at 62.23 38.1 0)
+			(hide yes)
+			(show_name no)
+			(do_not_autoplace no)
+			(effects
+				(font
+					(size 1.27 1.27)
+				)
+			)
+		)
+		(property "Datasheet" ""
+			(at 62.23 38.1 0)
+			(hide yes)
+			(show_name no)
+			(do_not_autoplace no)
+			(effects
+				(font
+					(size 1.27 1.27)
+				)
+			)
+		)
+		(property "Description" "Special symbol for telling ERC where power comes from"
+			(at 62.23 38.1 0)
+			(hide yes)
+			(show_name no)
+			(do_not_autoplace no)
+			(effects
+				(font
+					(size 1.27 1.27)
+				)
+			)
+		)
+		(pin "1"
+		)
+		(instances
+			(project "Motor_Driver"
+				(path "/73a47b03-d134-4703-ba74-88b80604f77f/44f57b88-633e-4540-abcf-a45c03b03b1e"
+					(reference "#FLG01")
+					(unit 1)
+				)
+			)
+		)
+	)
+	(symbol
 		(lib_id "Sensor_Temperature:TMP1075D")
 		(at 356.87 66.04 0)
@@
 			)
 		)
-		(property "Value" "C"
+		(property "Value" "100nF"
 			(at 165.1 104.14 90)
 			(show_name no)
@@
 			)
 		)
-		(property "Value" "C"
+		(property "Value" "100nF"
 			(at 302.26 46.99 90)
 			(show_name no)
@@
 			)
 		)
-		(property "Value" "C"
+		(property "Value" "100nF"
 			(at 165.1 140.97 90)
 			(show_name no)
@@
 	)
 	(symbol
+		(lib_id "power:PWR_FLAG")
+		(at 179.07 50.8 0)
+		(unit 1)
+		(body_style 1)
+		(exclude_from_sim no)
+		(in_bom yes)
+		(on_board yes)
+		(in_pos_files yes)
+		(dnp no)
+		(property "Reference" "#FLG03"
+			(at 179.07 48.895 0)
+			(hide yes)
+			(show_name no)
+			(do_not_autoplace no)
+			(effects
+				(font
+					(size 1.27 1.27)
+				)
+			)
+		)
+		(property "Value" "PWR_FLAG"
+			(at 181.864 46.736 0)
+			(show_name no)
+			(do_not_autoplace no)
+			(effects
+				(font
+					(size 1.27 1.27)
+				)
+			)
+		)
+		(property "Footprint" ""
+			(at 179.07 50.8 0)
+			(hide yes)
+			(show_name no)
+			(do_not_autoplace no)
+			(effects
+				(font
+					(size 1.27 1.27)
+				)
+			)
+		)
+		(property "Datasheet" ""
+			(at 179.07 50.8 0)
+			(hide yes)
+			(show_name no)
+			(do_not_autoplace no)
+			(effects
+				(font
+					(size 1.27 1.27)
+				)
+			)
+		)
+		(property "Description" "Special symbol for telling ERC where power comes from"
+			(at 179.07 50.8 0)
+			(hide yes)
+			(show_name no)
+			(do_not_autoplace no)
+			(effects
+				(font
+					(size 1.27 1.27)
+				)
+			)
+		)
+		(pin "1"
+		)
+		(instances
+			(project "Motor_Driver"
+				(path "/73a47b03-d134-4703-ba74-88b80604f77f/44f57b88-633e-4540-abcf-a45c03b03b1e"
+					(reference "#FLG03")
+					(unit 1)
+				)
+			)
+		)
+	)
+	(symbol
 		(lib_id "power:+12V")
 		(at 158.75 157.48 90)
@@
 			)
 		)
-		(property "Value" "C"
+		(property "Value" "100nF"
 			(at 347.98 46.99 90)
 			(show_name no)
